Commit message: 同步本地 src/：更新机器人与地图，纳入 community_person_16，整理目录结构
内容更新（虚拟机 ~/aic_ws/src 上的最新版本）：
- robot_description：CMakeLists.txt、urdf/robot.xacro、scripts/frame_remap.py、
  launch/{bringup,mapping,nav_bringup}.launch.py
- smart_community_gazebo/maps/community.{pgm,yaml}：重新建的图

新增：
- robot_description/scripts/explore_mapping.py
- smart_community_gazebo/models/community_person_16/（第 16 个人偶）

目录整理：此前误传到仓库根目录的 9 个包文件（CMakeLists.txt、package.xml、README.md、
TEAM_HANDOFF.md、VERSION.txt、launch_world.sh、layout_manifest.json、
person_manifest.csv、verify_project.sh）移入 smart_community_gazebo/，与 src/ 一致；
删除两个占位用的 .gitkeep。

其他：新增 .gitattributes 固定仓库换行为 LF；.gitignore 忽略 __pycache__ 等。
世界文件 worlds/smart_community_v2.sdf 内容不变（保持 include 引用的干净源文件版本）。

File: robot_description/urdf/robot.xacro (robot description, xacro)
@@ -13,9 +13,11 @@
   <xacro:property name="body_height" value="0.10"/>
   <xacro:property name="base_z" value="0.05"/>
+  <!-- base_footprint 是 TF 树的根（贴地面），base_link 挂在它上方 base_z 处。
+       顺序不能反：若 base_link 当根，KDL 会因「根节点带惯量」报警。 -->
   <link name="base_footprint"/>
   <joint name="base_footprint_joint" type="fixed">
-    <parent link="base_link"/>
-    <child link="base_footprint"/>
-    <origin xyz="0 0 -${base_z}" rpy="0 0 0"/>
+    <parent link="base_footprint"/>
+    <child link="base_link"/>
+    <origin xyz="0 0 ${base_z}" rpy="0 0 0"/>
   </joint>
   <link name="base_link">
@@ -48,5 +50,6 @@
       </visual>
       <collision>
-        <geometry><sphere radius="${wheel_radius}"/></geometry>
+        <origin xyz="0 0 0" rpy="1.5708 0 0"/>
+        <geometry><cylinder radius="${wheel_radius}" length="${wheel_width}"/></geometry>
       </collision>
     </link>
@@ -141,4 +144,9 @@
     </plugin>
   </gazebo>
+  <!-- gz-sim 8 的 IMU 不由 sensors-system 处理，必须显式加载 imu-system 插件，
+       否则 <sensor type="imu"> 会被静默丢弃、`gz topic -l` 里根本没有 /imu。 -->
+  <gazebo>
+    <plugin filename="gz-sim-imu-system" name="gz::sim::systems::Imu"/>
+  </gazebo>
   <gazebo reference="lidar_link">
     <sensor name="lidar" type="gpu_lidar">
@@ -161,5 +169,5 @@
       </lidar>
       <always_on>1</always_on>
-      <update_rate>10</update_rate>
+      <update_rate>30</update_rate>
       <topic>lidar</topic>
     </sensor>
