Commit message: 世界自带车 + 修正轮轴符号：前进方向与车头一致
- worlds/smart_community_v2.sdf：保留世界内置的 patrol_bot（手工加的，停在起点板
  3.88/3.88），并入缩短后的停车区路沿（curb_v_parking_left 长度 4.2→3.6、
  中心 y 2.1→1.7904，让出顶边道路的口子，小车才开得出去）；
  烘焙车的轮轴 0 -1 0 → 0 1 0，位姿归到 x=3.88 y=3.88 yaw=π
- robot.xacro：轮轴 axis 0 -1 0 → 0 1 0。原有写法会让 gz 的 DiffDrive 把
  linear.x>0 解释成沿模型 -X 走，小车“倒着走”，前进方向与车头（相机在 +X）相反
- spawn_robot.launch.py：新增 spawn 参数（默认 true），默认起点仍为
  x/y=3.88、yaw=π（朝西）
- bringup / nav_bringup / mapping：传 spawn:=false，世界自带车时只起
  robot_state_publisher，不再重复 spawn（同名撞名会让 x/y/yaw 参数静默失效）

实测（headless）：世界内 patrol_bot 恰好 1 个，位于 (3.88, 3.88) yaw=π；
发 linear.x=+0.15 后 x 由 3.88 变 3.363（往西），y 与 yaw 不变，
顺利穿过缩短路沿留出的缺口。

File: src/robot_description/urdf/robot.xacro (robot description, xacro)
@@ -58,5 +58,7 @@
       <child link="${name}"/>
       <origin xyz="0.04 ${y_pos} 0" rpy="0 0 0"/>
-      <axis xyz="0 -1 0"/>
+      <!-- 轮轴必须指向 +Y：指向 -Y 会让 gz 的 DiffDrive 把 linear.x>0 解释成往 -X 走，
+           小车就会“倒着走”（前进方向与车头相反，相机装在 +X 侧）。 -->
+      <axis xyz="0 1 0"/>
     </joint>
     <gazebo reference="${name}">
